Commit message: working gazebo

File: vbn_ml/urdf/realsense.urdf.xacro (robot description, xacro)
@@ -15,5 +15,5 @@
   <gazebo reference="front_realsense">
     <turnGravityOff>true</turnGravityOff>
-    <sensor type="depth" name="front_realsense_depth">
+    <sensor name="front_camera" type="camera">
       <update_rate>30</update_rate>
       <camera>
@@ -32,27 +32,7 @@
         </clip>
       </camera>
-      <plugin name="kinect_controller" filename="libgazebo_ros_openni_kinect.so">
-        <baseline>0.2</baseline>
-        <alwaysOn>true</alwaysOn>
-        <updateRate>30</updateRate>
-        <cameraName>realsense</cameraName>
-        <imageTopicName>color/image_raw</imageTopicName>
-        <cameraInfoTopicName>color/camera_info</cameraInfoTopicName>
-        <depthImageTopicName>depth/image_rect_raw</depthImageTopicName>
-        <depthImageInfoTopicName>depth/camera_info</depthImageInfoTopicName>
-        <pointCloudTopicName>depth/color/points</pointCloudTopicName>
-        <frameName>front_realsense_gazebo</frameName>
-        <pointCloudCutoff>0.105</pointCloudCutoff>
-        <pointCloudCutoffMax>8.0</pointCloudCutoffMax>
-        <distortionK1>0.00000001</distortionK1>
-        <distortionK2>0.00000001</distortionK2>
-        <distortionK3>0.00000001</distortionK3>
-        <distortionT1>0.00000001</distortionT1>
-        <distortionT2>0.00000001</distortionT2>
-        <CxPrime>0</CxPrime>
-        <Cx>0</Cx>
-        <Cy>0</Cy>
-        <focalLength>0</focalLength>
-        <hackBaseline>0</hackBaseline>
+      <plugin name="camera_plugin" filename="libgazebo_ros_camera.so">
+        <alwaysOn>1</alwaysOn>
+         <updateRate>0</updateRate>
       </plugin>
     </sensor>
@@ -62,5 +42,5 @@
       <origin xyz="0.02 0 0" rpy="${pi/2} 0 ${pi/2}" />
       <geometry>
-        <mesh filename="package://realsense2_description/meshes/d435.dae" />
+        <mesh filename="file:///home/olagh/ros_ml_ws/src/realsense-ros/realsense2_description/meshes/d435.dae" />
       </geometry>
       <material name="white" />
